File: Projects/Toy Design/.history/Toy Design.kicad_pcb (KiCad board)
At the start: 2 copper layers, 170 x 120 mm, 92 parts, among them J1 Conn_01x01_Pin, J2 Conn_01x01_Pin, J3 FTSH-107-01-X-DV-K-TR, SW1 5GTH935, SW2 5GTH935, U1 TLV61048DBVR, U10 STM32G030K6T6, U11 MCP3208-CI/SL, U12 74HC595, U13 74HC595, U14 74HC595, U15 74HC595, U16 74HC595, U17 74HC595, U2 MCP73123, U3 NCP1117-5.0_SOT223, U4 MLX90333, U5 A1330, U6 A1330, U7 NCP1117-3.3_SOT223, U8 A1330, U9 TXU0104

Commit message: Update into ordering
Parts:
- R4: value 601k -> 675k
- moved R41 87.1 mm to (158.5, 34.5), turned to 180 degrees
- moved R43 23.2 mm to (190.8, 34.5), turned to 180 degrees
- moved R42 17.3 mm to (175.5, 34.5), turned to 180 degrees
Connections:
- net +5.6V renamed +6.2
- U9 pad 3: unconnected-(U9-A2-Pad3) -> GND
Routing:
- net Net-(U10-PA7): track 0.00 -> 103.7 mm, vias 0 -> 2
- net Net-(U10-PA8): track 0.00 -> 82.3 mm, vias 0 -> 2
- net Net-(U10-PA9/PA11): track 0.00 -> 77.2 mm
- net +3.3V: track 395.8 -> 438.4 mm, vias 7 -> 9
- net Net-(D4-K): track 0.00 -> 5.75 mm
- net ~{OE}: track 232.6 -> 238.2 mm
- net Net-(U13-SER): track 87.4 -> 93.0 mm
- net Net-(D5-K): track 0.00 -> 3.75 mm
- net Net-(D6-K): track 0.00 -> 3.50 mm
- net GND: track 55.4 -> 58.1 mm, vias 260 -> 261
