File: Projects/Toy Design/.history/Toy Design.kicad_sch (KiCad schematic)
At the start: 48 parts, among them J1 Conn_01x01_Pin, J2 Conn_01x01_Pin, J3 FTSH-107-01-X-DV-K-TR, SW1 5GTH935, SW2 5GTH935, U1 TLV61048DBVR, U10 STM32G030K6T6, U11 MCP3208-CI/SL, U2 MCP73123, U3 NCP1117-5.0_SOT223, U4 MLX90333, U5 A1330, U6 A1330, U7 NCP1117-3.3_SOT223, U8 A1330, U9 TXU0104

Commit message: Finalzied DRCs Added 3 LEDs
Parts:
- added C16: 10uF, Capacitor_SMD:C_1206_3216Metric_Pad1.33x1.80mm_HandSolder, symbol Device:C
- added D5, D6: LED, LED_THT:LED_D5.0mm, symbol Device:LED
- added R42, R43: 650, Resistor_SMD:R_0805_2012Metric_Pad1.20x1.40mm_HandSolder, symbol Device:R_US
Connections:
- net +3.3V: now also D5.2 (A), D6.2 (A)
- net GND: now also C16.2
- net at D1.1 (K), D2.1 (K), L1.1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: now also C16.1
- net ~{OE}: now reaches U10.1 (PB9)
- net at U10.18 (PA8): now also R42.2
- net at U10.22 (PA9/PA11): now also R43.2
- new net: D5.1 (K), R42.1
- new net: D6.1 (K), R43.1

Commit message: Update into ordering
Parts:
- R4: value 601k -> 675k
Connections:
- net GND: now also U9.3 (A2)
- net +5.6V renamed +6.2
Changed lines of the file:
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@@
 	(wire
 		(pts
+			(xy 265.43 179.07) (xy 261.62 179.07)
+		)
+		(stroke
+			(width 0)
+			(type default)
+		)
+	)
+	(wire
+		(pts
 			(xy 60.96 58.42) (xy 60.96 55.88)
 		)
@@
 	(wire
 		(pts
+			(xy 261.62 179.07) (xy 261.62 180.34)
+		)
+		(stroke
+			(width 0)
+			(type default)
+		)
+	)
+	(wire
+		(pts
+			(xy 261.62 180.34) (xy 259.08 180.34)
+		)
+		(stroke
+			(width 0)
+			(type default)
+		)
+	)
+	(wire
+		(pts
 			(xy 242.57 107.95) (xy 242.57 110.49)
 		)
@@
 			)
 		)
-		(property "Value" "601k"
+		(property "Value" "675k"
 			(at 170.18 45.7199 0)
 			(show_name no)
@@
 			)
 		)
-		(property "Value" "+5.6V"
-			(at 167.64 31.75 0)
+		(property "Value" "+6.2"
+			(at 170.18 35.5599 0)
 			(show_name no)
 			(do_not_autoplace no)
@@
 					(size 1.27 1.27)
 				)
+				(justify left)
 			)
 		)
@@
 					(unit 1)
 				)
+			)
+		)
+	)
+	(symbol
+		(lib_id "power:GND")
+		(at 265.43 179.07 0)
+		(unit 1)
+		(body_style 1)
+		(exclude_from_sim no)
+		(in_bom yes)
+		(on_board yes)
+		(in_pos_files yes)
+		(dnp no)
+		(property "Reference" "#PWR070"
+			(at 265.43 185.42 0)
+			(hide yes)
+			(show_name no)
+			(do_not_autoplace no)
+			(effects
+				(font
+					(size 1.27 1.27)
+				)
+			)
+		)
+		(property "Value" "GND"
+			(at 269.24 180.594 0)
+			(show_name no)
+			(do_not_autoplace no)
+			(effects
+				(font
+					(size 1.27 1.27)
+				)
+			)
+		)
+		(property "Footprint" ""
+			(at 265.43 179.07 0)
+			(hide yes)
+			(show_name no)
+			(do_not_autoplace no)
+			(effects
+				(font
+					(size 1.27 1.27)
+				)
+			)
+		)
+		(property "Datasheet" ""
+			(at 265.43 179.07 0)
+			(hide yes)
+			(show_name no)
+			(do_not_autoplace no)
+			(effects
+				(font
+					(size 1.27 1.27)
+				)
+			)
+		)
+		(property "Description" "Power symbol creates a global label with name \"GND\" , ground"
+			(at 265.43 179.07 0)
+			(hide yes)
+			(show_name no)
+			(do_not_autoplace no)
+			(effects
+				(font
+					(size 1.27 1.27)
+				)
+			)
+		)
+		(pin "1"
+		)
+		(instances
+			(project "Toy Design"
+				(path "/c85456d0-c9f8-47a9-8124-8a5f769becea"
+					(reference "#PWR070")
+					(unit 1)
+				)
